Commit message: Mount HandUMI rotated 180 deg on flange; tabletop 4 mm above base

File: src/kuka_sim/assets/iiwa7_handumi/iiwa7_handumi.urdf (robot description, URDF)
Before this commit: robot lbr_iiwa7_r800, 24 links, 23 joints
Joints:
- joint gripper_flange__gripper: origin xyz=0 0 0 rpy=0 0 0 -> xyz=0 0 0 rpy=0 0 3.14159265

Commit message: Render from gripper-aware calibration; media flange, colours, wood table; compare tools

File: src/kuka_sim/assets/iiwa7_handumi/iiwa7_handumi.urdf (robot description, URDF)
Before this commit: robot lbr_iiwa7_r800, 24 links, 23 joints
Links:
- link gripper_assembly_root: geometry collision cylinder length=0.022 radius=0.04; visual cylinder length=0.022 radius=0.04
Joints:
- joint gripper_flange__gripper: origin xyz=0 0 0 rpy=0 0 3.14159265 -> xyz=0 0 0.022 rpy=0 0 3.14159265
